File: kicad/musicbox/musicbox.kicad_sch (KiCad schematic)
At the start: 8 parts

Commit message: Updated the documentation
Parts:
- removed LED3: ~, symbol custom_parts:WS2812B
Connections:
- new net: LED1. (VIN), LED2. (VIN)
- no-connect marks 12 -> 11
Other:
- moved on the sheet: Audioboard, BT1, LS1, LS2

Commit message: Working on newer prototype
Parts:
- removed Audioboard: ~, symbol custom_parts:AiThinker_ESP32_AudioKit
- removed LS2: Speaker, symbol Device:Speaker
- added ESP32: ~, symbol custom_parts:ESP32_DevKitC
- added MAX98357A: ~, symbol custom_parts:MAX98357A
- added Next, Prev, Start/Stop: Button, symbol Switch:SW_Push
- added SDCardReader: ~, symbol custom_parts:SDCardReader
Connections:
- net 3V3: now also ESP32. (GPIO06), Next.2, Prev.2, SDCardReader.5 (VCC), Start/Stop.2
- net ADR_LED: now also ESP32. (GPIO06)
- net GND: now also ESP32. (GPIO06), MAX98357A.2 (GND), MAX98357A.4 (GAIN), SDCardReader.6 (GND)
- net I2C_SCL: now also ESP32. (GPIO06)
- net I2C_SDA: now also ESP32. (GPIO06)
- net RFID_RST: now also ESP32. (GPIO06)
- net VBAT: now also MAX98357A.1 (VIN)
- net at LS1.1: now also MAX98357A. (SPK-)
- net at LS1.2: now also MAX98357A. (SPK-)
- new net: LED1. (DOUT), LED2. (DOUT)
- new net BT1: ESP32. (GPIO06), Start/Stop.1
- new net BT2: ESP32. (GPIO06), Prev.1
- new net BT3: ESP32. (GPIO06), Next.1
- new net I2S_BCK: ESP32. (GPIO06), MAX98357A.6 (BCLK)
- new net I2S_DIN: ESP32. (GPIO06), MAX98357A.5 (DIN)
- new net I2S_WS: ESP32. (GPIO06), MAX98357A.7 (LRC)
- new net RFID_IRQ: ESP32. (GPIO06), RFIDReader. (GND)
- new net SPI_CLK: ESP32. (GPIO06), SDCardReader.2 (CLK)
- new net SPI_MISO: ESP32. (GPIO06), SDCardReader.4 (MISO)
- new net SPI_MOSI: ESP32. (GPIO06), SDCardReader.3 (MOSI)
- new net SPI_SS: ESP32. (GPIO06), SDCardReader.1 (CS)
- no-connect marks 11 -> 10
Other:
- note added: "Audio Output"
- note added: "Buttons / Controls"
- note added: "ESP32 Microcontroller"
- note added: "Power management"
- note added: "RFID interface"
- note added: "Storage"
- note removed: "Key4 == Start / Stop Key5 == Prev / Vol - Key6 == Next / Vol +"
- note removed: "SD is running in 1bit Mode CLK = GPIO14 CMD = GPIO15 D0 = GPIO02"
- moved on the sheet: BT1, LS1, RFIDReader

Commit message: Working on newer prototype
Parts:
- added BK1: ~, symbol custom_parts:BuckConverter
- added CHG1: ~, symbol custom_parts:USBLiPo
- added SW1: SW, symbol Switch:SW_DPST_x2
- renumbered MAX98357A to AMP, SDCardReader to RD1, RFIDReader to RF1
Connections:
- net 3V3: now also BK1. (GO)
- net GND: now also BK1. (GO); no longer BT1.2 (-)
- net VBAT: now also BK1. (GO), SW1.2 (B); no longer BT1.1 (+)
- new net: LED1. (DOUT), LED2. (DOUT)
- new net BAT+: BT1.1 (+), CHG1. (B-), SW1.1 (A)
- new net BAT-: BK1. (GO), BT1.2 (-), CHG1. (B-)
- no-connect marks 10 -> 21
Other:
- note added: "The ESP32 IO Pins must be configures as INPUT_PULL_DOWN."
- moved on the sheet: BT1, Next, Prev, Start/Stop

Commit message: Working on ewer version
Connections:
- net SPI_CLK renamed SPI_SCK
- new net: LED1. (DOUT), LED2. (DOUT)
Other:
- note added: "The ESP32 IO Pins must be configures as INPUT_PULLDOWN"
- note removed: "The ESP32 IO Pins must be configures as INPUT_PULL_DOWN."
- moved on the sheet: Next, Prev, Start/Stop
Changed lines of the file:
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@@
 		)
 	)
-	(text "The ESP32 IO Pins\nmust be configures\nas INPUT_PULL_DOWN."
+	(text "The ESP32 IO Pins\nmust be configures\nas INPUT_PULLDOWN"
 		(exclude_from_sim no)
 		(at 149.86 95.758 0)
@@
 	)
 	(junction
-		(at 189.23 92.71)
+		(at 187.96 91.44)
 		(diameter 0)
 		(color 0 0 0 0)
 	)
 	(junction
-		(at 189.23 85.09)
+		(at 187.96 83.82)
 		(diameter 0)
 		(color 0 0 0 0)
@@
 	)
 	(no_connect
-		(at 134.62 44.45)
-	)
-	(no_connect
 		(at 96.52 64.77)
 	)
@@
 		(at 96.52 52.07)
 	)
+	(no_connect
+		(at 134.62 46.99)
+	)
 	(wire
 		(pts
@@
 	(wire
 		(pts
-			(xy 182.88 92.71) (xy 189.23 92.71)
+			(xy 181.61 91.44) (xy 187.96 91.44)
 		)
 		(stroke
@@
 	(wire
 		(pts
-			(xy 182.88 85.09) (xy 189.23 85.09)
+			(xy 181.61 83.82) (xy 187.96 83.82)
 		)
 		(stroke
@@
 	(wire
 		(pts
-			(xy 182.88 100.33) (xy 189.23 100.33)
+			(xy 181.61 99.06) (xy 187.96 99.06)
 		)
 		(stroke
@@
 	(wire
 		(pts
-			(xy 189.23 85.09) (xy 189.23 92.71)
+			(xy 187.96 83.82) (xy 187.96 91.44)
 		)
 		(stroke
@@
 	(wire
 		(pts
-			(xy 189.23 100.33) (xy 189.23 92.71)
+			(xy 187.96 99.06) (xy 187.96 91.44)
 		)
 		(stroke
@@
 	(wire
 		(pts
-			(xy 189.23 82.55) (xy 189.23 85.09)
+			(xy 187.96 81.28) (xy 187.96 83.82)
 		)
 		(stroke
@@
 		)
 	)
-	(label "SPI_SS"
-		(at 134.62 46.99 0)
-		(effects
-			(font
-				(size 1.27 1.27)
-			)
-			(justify left bottom)
-		)
-	)
 	(label "I2C_SCL"
 		(at 54.61 40.64 180)
@@
 	)
 	(label "BT1"
-		(at 172.72 85.09 180)
+		(at 171.45 83.82 180)
 		(effects
 			(font
@@
 	)
 	(label "BT3"
-		(at 172.72 100.33 180)
+		(at 171.45 99.06 180)
 		(effects
 			(font
@@
 		)
 	)
-	(label "SPI_CLK"
+	(label "SPI_SCK"
 		(at 97.79 87.63 180)
 		(effects
@@
 		)
 	)
+	(label "SPI_SS"
+		(at 134.62 44.45 0)
+		(effects
+			(font
+				(size 1.27 1.27)
+			)
+			(justify left bottom)
+		)
+	)
 	(label "SPI_MOSI"
 		(at 97.79 90.17 180)
@@
 	)
 	(label "BT2"
-		(at 172.72 92.71 180)
+		(at 171.45 91.44 180)
 		(effects
 			(font
@@
 		)
 	)
-	(label "SPI_CLK"
+	(label "SPI_SCK"
 		(at 134.62 41.91 0)
 		(effects
@@
 	(symbol
 		(lib_id "Switch:SW_Push")
-		(at 177.8 100.33 0)
+		(at 176.53 99.06 0)
 		(unit 1)
 		(exclude_from_sim no)
@@
 		(dnp no)
 		(property "Reference" "Next"
-			(at 177.292 96.266 0)
+			(at 176.022 94.996 0)
 			(effects
 				(font
@@
 		)
 		(property "Value" "Button"
-			(at 177.8 95.25 0)
-			(effects
-				(font
-					(size 1.27 1.27)
-				)
-				(hide yes)
-			)
-		)
-		(property "Footprint" ""
-			(at 177.8 95.25 0)
+			(at 176.53 93.98 0)
+			(effects
+				(font
+					(size 1.27 1.27)
+				)
+				(hide yes)
+			)
+		)
+		(property "Footprint" ""
+			(at 176.53 93.98 0)
 			(effects
 				(font
@@
 		)
 		(property "Datasheet" "~"
-			(at 177.8 95.25 0)
+			(at 176.53 93.98 0)
 			(effects
 				(font
@@
 		)
 		(property "Description" "Push button switch, generic, two pins"
-			(at 177.8 100.33 0)
+			(at 176.53 99.06 0)
 			(effects
 				(font
@@
 	(symbol
 		(lib_id "Switch:SW_Push")
-		(at 177.8 92.71 0)
+		(at 176.53 91.44 0)
 		(unit 1)
 		(exclude_from_sim no)
@@
 		(dnp no)
 		(property "Reference" "Prev"
-			(at 177.292 88.646 0)
+			(at 176.022 87.376 0)
 			(effects
 				(font
@@
 		)
 		(property "Value" "Button"
-			(at 177.8 87.63 0)
-			(effects
-				(font
-					(size 1.27 1.27)
-				)
-				(hide yes)
-			)
-		)
-		(property "Footprint" ""
-			(at 177.8 87.63 0)
+			(at 176.53 86.36 0)
+			(effects
+				(font
+					(size 1.27 1.27)
+				)
+				(hide yes)
+			)
+		)
+		(property "Footprint" ""
+			(at 176.53 86.36 0)
 			(effects
 				(font
@@
 		)
 		(property "Datasheet" "~"
-			(at 177.8 87.63 0)
+			(at 176.53 86.36 0)
 			(effects
 				(font
@@
 		)
 		(property "Description" "Push button switch, generic, two pins"
-			(at 177.8 92.71 0)
+			(at 176.53 91.44 0)
 			(effects
 				(font
@@
 	)
 	(symbol
-		(lib_name "WS2812B_1")
 		(lib_id "custom_parts:WS2812B")
 		(at 59.69 92.71 0)
@@
 	)
 	(symbol
+		(lib_name "WS2812B_1")
 		(lib_id "custom_parts:WS2812B")
 		(at 34.29 92.71 0)
@@
 	(symbol
 		(lib_id "power:+5V")
-		(at 189.23 82.55 0)
+		(at 187.96 81.28 0)
 		(unit 1)
 		(exclude_from_sim no)
@@
 		(dnp no)
 		(property "Reference" "#PWR016"
-			(at 189.23 86.36 0)
+			(at 187.96 85.09 0)
 			(effects
 				(font
@@
 		)
 		(property "Value" "3V3"
-			(at 189.23 78.994 0)
-			(effects
-				(font
-					(size 1.27 1.27)
-				)
-			)
-		)
-		(property "Footprint" ""
-			(at 189.23 82.55 0)
+			(at 187.96 77.724 0)
+			(effects
+				(font
+					(size 1.27 1.27)
+				)
+			)
+		)
+		(property "Footprint" ""
+			(at 187.96 81.28 0)
 			(effects
 				(font
@@
 		)
 		(property "Datasheet" ""
-			(at 189.23 82.55 0)
+			(at 187.96 81.28 0)
 			(effects
 				(font
@@
 		)
 		(property "Description" "Power symbol creates a global label with name \"+5V\""
-			(at 189.23 82.55 0)
+			(at 187.96 81.28 0)
 			(effects
 				(font
@@
 	(symbol
 		(lib_id "Switch:SW_Push")
-		(at 177.8 85.09 0)
+		(at 176.53 83.82 0)
 		(unit 1)
 		(exclude_from_sim no)
@@
 		(dnp no)
 		(property "Reference" "Start/Stop"
-			(at 177.292 81.026 0)
+			(at 176.022 79.756 0)
 			(effects
 				(font
@@
 		)
 		(property "Value" "Button"
-			(at 177.8 80.01 0)
-			(effects
-				(font
-					(size 1.27 1.27)
-				)
-				(hide yes)
-			)
-		)
-		(property "Footprint" ""
-			(at 177.8 80.01 0)
+			(at 176.53 78.74 0)
+			(effects
+				(font
+					(size 1.27 1.27)
+				)
+				(hide yes)
+			)
+		)
+		(property "Footprint" ""
+			(at 176.53 78.74 0)
 			(effects
 				(font
@@
 		)
 		(property "Datasheet" "~"
-			(at 177.8 80.01 0)
+			(at 176.53 78.74 0)
 			(effects
 				(font
@@
 		)
 		(property "Description" "Push button switch, generic, two pins"
-			(at 177.8 85.09 0)
-			(effects
-				(font
+			(at 176.53 83.82 0)
+			(effects
+				(font

Commit message: Bug fixing
Connections:
- new net: LED1. (DOUT), LED2. (DOUT)
Changed lines of the file:
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@@
+	)
+	(no_connect
+		(at 96.52 31.75)
 	)
 	(no_connect
@@
 	)
 	(no_connect
+		(at 96.52 26.67)
+	)
+	(no_connect
 		(at 162.56 29.21)
 	)
@@
 	)
 	(no_connect
-		(at 134.62 49.53)
-	)
-	(no_connect
 		(at 134.62 67.31)
 	)
@@
 	)
 	(no_connect
-		(at 134.62 52.07)
-	)
-	(no_connect
 		(at 134.62 64.77)
 	)
@@
 	)
 	(no_connect
-		(at 134.62 46.99)
+		(at 96.52 29.21)
 	)
 	(wire
@@
 		)
 	)
-	(label "BT3"
-		(at 96.52 31.75 180)
-		(effects
-			(font
-				(size 1.27 1.27)
-			)
-			(justify right bottom)
+	(label "BT2"
+		(at 134.62 49.53 0)
+		(effects
+			(font
+				(size 1.27 1.27)
+			)
+			(justify left bottom)
 		)
 	)
@@
 	)
 	(label "BT3"
+		(at 134.62 46.99 0)
+		(effects
+			(font
+				(size 1.27 1.27)
+			)
+			(justify left bottom)
+		)
+	)
+	(label "BT3"
 		(at 171.45 99.06 180)
 		(effects
@@
 		)
 	)
+	(label "BT1"
+		(at 134.62 52.07 0)
+		(effects
+			(font
+				(size 1.27 1.27)
+			)
+			(justify left bottom)
+		)
+	)
 	(label "ADR_LED"
 		(at 96.52 41.91 180)
@@
 		)
 	)
-	(label "BT1"
-		(at 96.52 26.67 180)
-		(effects
-			(font
-				(size 1.27 1.27)
-			)
-			(justify right bottom)
-		)
-	)
 	(label "RFID_IRQ"
 		(at 54.61 45.72 180)
@@
 		(effects
 			(font
-				(size 1.27 1.27)
-			)
-			(justify right bottom)
-		)
-	)
-	(label "BT2"
-		(at 96.52 29.21 180)
-		(effects
-			(font

Commit message: Bug fixing
Parts:
- removed LS1: Speaker, symbol Device:Speaker
- added BT1Con1, BT2Con1, BT3Con1, PWRCon1: ~, Connector_JST:JST_PH_B2B-PH-K_1x02_P2.00mm_Vertical, symbol Connector:Conn_01x02_Socket
- added IO1: IO, CustomFootprints:Pads_2x10, symbol Connector_Generic:Conn_02x10_Top_Bottom
- added NeoPixelCon1: ~, Connector_JST:JST_PH_B3B-PH-K_1x03_P2.00mm_Vertical, symbol Connector:Conn_01x03_Socket
- added RFIDCon1: Conn_01x06_Socket, Connector_JST:JST_PH_B6B-PH-K_1x06_P2.00mm_Vertical, symbol Connector:Conn_01x06_Socket
- AMP1: renamed from AMP; footprint (none) -> CustomFootprints:MAX98357A
- ESP32: footprint (none) -> CustomFootprints:ESP32DevKit
- RD1: footprint (none) -> CustomFootprints:SDCardReader
- renumbered Next to Next1, Prev to Prev1, Start/Stop to Start/Stop1
Connections:
- net 3V3: now also BK1.2 (VO), ESP32.1 (3V3), RD1.1 (VCC), RF1.1 (VCC), BT1Con1.2 (Pin_2), BT2Con1.2 (Pin_2), BT3Con1.2 (Pin_2), IO1.18 (Pin_18), NeoPixelCon1.1 (Pin_1), PWRCon1.1 (Pin_1), RFIDCon1.5 (Pin_5); no longer BK1. (GO), ESP32. (GPIO06), RD1.5 (VCC), RF1. (GND)
- net ADR_LED: now also ESP32.9 (GPIO25), LED1.1 (DIN), NeoPixelCon1.2 (Pin_2); no longer ESP32. (GPIO06), LED1. (DOUT)
- net BAT+: now also CHG1.1 (B+); no longer CHG1. (B-)
- net BT1: now also ESP32.32 (GPIO04), BT1Con1.1 (Pin_1); no longer ESP32. (GPIO06)
- net BT2: now also ESP32.31 (GPIO16), BT2Con1.1 (Pin_1); no longer ESP32. (GPIO06)
- net BT3: now also ESP32.30 (GPIO17), BT3Con1.1 (Pin_1); no longer ESP32. (GPIO06)
- net GND: now also AMP1.6 (GND), BK1.3 (GI), BK1.4 (GO), BT1.2 (-), CHG1.2 (B-), ESP32.14 (GND), ESP32.20 (GND), ESP32.26 (GND), LED1.3 (GND), LED2.3 (GND), RF1.6 (GND), NeoPixelCon1.3 (Pin_3), PWRCon1.2 (Pin_2), RFIDCon1.6 (Pin_6); no longer AMP1.2 (GND), BK1. (GO), ESP32. (GPIO06), LED1. (DOUT), LED2. (DOUT), RF1. (GND)
- net I2C_SCL: now also ESP32.22 (GPIO22), RF1.3 (SCL), RFIDCon1.2 (Pin_2); no longer ESP32. (GPIO06), RF1. (GND)
- net I2C_SDA: now also ESP32.25 (GPIO21), RF1.2 (SDA), RFIDCon1.1 (Pin_1); no longer ESP32. (GPIO06), RF1. (GND)
- net I2S_BCK: now also AMP1.2 (BCLK), ESP32.10 (GPIO26); no longer AMP1.6 (BCLK), ESP32. (GPIO06)
- net I2S_DIN: now also AMP1.3 (DIN), ESP32.11 (GPIO27); no longer AMP1.5 (DIN), ESP32. (GPIO06)
- net I2S_WS: now also AMP1.1 (LRC), ESP32.12 (GPIO14); no longer AMP1.7 (LRC), ESP32. (GPIO06)
- net RFID_IRQ: now also ESP32.7 (GPIO32), RF1.4 (IRQ), RFIDCon1.3 (Pin_3); no longer ESP32. (GPIO06), RF1. (GND)
- net RFID_RST: now also ESP32.8 (GPIO33), RF1.5 (RST), RFIDCon1.4 (Pin_4); no longer ESP32. (GPIO06), RF1. (GND)
- net SPI_MISO: now also ESP32.27 (GPIO19), RD1.5 (MISO); no longer ESP32. (GPIO06), RD1.4 (MISO)
- net SPI_MOSI: now also ESP32.21 (GPIO23); no longer ESP32. (GPIO06)
- net SPI_SCK: now also ESP32.28 (GPIO18), RD1.4 (SCK); no longer ESP32. (GPIO06), RD1.2 (SCK)
- net SPI_SS: now also ESP32.29 (GPIO05), RD1.2 (CS); no longer ESP32. (GPIO06), RD1.1 (CS)
- net VBAT: now also AMP1.7 (VIN), BK1.1 (VI), LED1.2 (VIN), LED2.2 (VIN); no longer AMP1.1 (VIN), BK1. (GO), LED1. (DOUT), LED2. (DOUT)
- removed net BAT-: BK1. (GO), BT1.2 (-), CHG1. (B-)
- new net: LED1.4 (DOUT), LED2.1 (DIN)
- new net GPIO00: ESP32.33 (GPIO00), IO1.11 (Pin_11)
- new net GPIO01: ESP32.23 (GPIO01), IO1.9 (Pin_9)
- new net GPIO02: ESP32.34 (GPIO02), IO1.12 (Pin_12)
- new net GPIO03: ESP32.24 (GPIO03), IO1.10 (Pin_10)
- new net GPIO06: ESP32.38 (GPIO06), IO1.16 (Pin_16)
- new net GPIO07: ESP32.37 (GPIO07), IO1.15 (Pin_15)
- new net GPIO08: ESP32.36 (GPIO08), IO1.14 (Pin_14)
- new net GPIO09: ESP32.16 (GPIO09), IO1.7 (Pin_7)
- new net GPIO10: ESP32.17 (GPIO10), IO1.8 (Pin_8)
- new net GPIO11: ESP32.18 (GPIO11)
- new net GPIO12: ESP32.13 (GPIO12), IO1.5 (Pin_5)
- new net GPIO13: ESP32.15 (GPIO13), IO1.6 (Pin_6)
- new net GPIO15: ESP32.35 (GPIO15), IO1.13 (Pin_13)
- new net GPIO34: ESP32.5 (GPIO34), IO1.3 (Pin_3)
- new net GPIO35: ESP32.6 (GPIO35), IO1.4 (Pin_4)
- new net GPIO36: ESP32.3 (GPIO36), IO1.1 (Pin_1)
- new net GPIO39: ESP32.4 (GPIO39), IO1.2 (Pin_2)
- new net RST: ESP32.2 (RESET), IO1.17 (Pin_17)
- no-connect marks 21 -> 5
Other:
- note added: "Additional I/O"
- note added: "The ESP32 IO Pins must be configures as INPUT_PULLDOWN PCB only includes Button connectors!"
- note removed: "The ESP32 IO Pins must be configures as INPUT_PULLDOWN"
- moved on the sheet: Next1, Prev1, Start/Stop1
